File: rotor_power_5Vx4/pcb_kamex_fuentes_5v_7amp_1.0.brd (EAGLE design)
At the start: 79 x 60 mm, 56 parts, among them IC1 MAX20008AFOC_VY+T, IC2 MAX20008AFOC_VY+T, IC3 MAX20008AFOC_VY+T, IC4 MAX20008AFOC_VY+T

Commit message: Cambios Juan Carlos
Parts:
- moved 0,1UF12 73.7 mm to (123.1, 21.2), turned to 0 degrees
- moved NO_CONNECT3 69.4 mm to (123.2, 25.0), turned to 0 degrees
- moved 12K3 68.6 mm to (117.8, 22.2), turned to 270 degrees
- moved 2,2UF4 67.0 mm to (115.4, 22.2), turned to 270 degrees
- moved 22,UF8 66.8 mm to (125.7, 29.5), turned to 90 degrees
- moved 1NF3 65.4 mm to (112.8, 22.2), turned to 90 degrees
- moved 22,UF7 64.7 mm to (123.5, 29.5), turned to 90 degrees
- moved 22K3 62.9 mm to (109.7, 22.8), turned to 270 degrees
- moved 0,1UF10 62.5 mm to (121.1, 29.6), turned to 270 degrees
- moved IC4 59.3 mm to (116.2, 28.9), turned to 180 degrees
- moved 4.7PF3 58.9 mm to (106.4, 24.7), turned to 90 degrees
- moved 0,1UF11 58.0 mm to (112.0, 27.6), turned to 90 degrees
- moved 4,7UF.4 56.7 mm to (109.8, 27.6), turned to 90 degrees
- moved L4 47.6 mm to (116.3, 39.3), turned to 90 degrees
- moved 12K2 1.02 mm to (52.6, 12.4)
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