File: zenit_main/pcb_khamex_zenit_V0.1_rev_5.3.sch (EAGLE design)
At the start: 49 parts, among them IC1 PCA9306JKZ, IC2 SN65HVD230DR, J2 52559-2253, J3 686110188622, J4 686110188622, J5 612010235121, U1 AMS1117-1.8

Commit message: Cambios Juan Carlos
Parts:
- removed 5V_MPU, GND_ROTOR, GND_ROTOR1, GND_ROTOR2, GND_ROTOR3: SE14, solpad:SE14
- added GND_OPI, GND_SERVOS, LIGHTS_GND: SE14, solpad:SE14
- renumbered J5 to J1
Connections:
- removed net 5V_MPUS: 5V_CARCASA.MP, 5V_MPU.MP
- removed net GND: J1.10, J1.5, J1.7
- removed net GND_PLANE: 10K_GND.2, C4.1, C5.1, GND_CARCASA.MP, GND_LIDAR.P, GND_ROTOR.MP, GND_ROTOR1.MP, GND_ROTOR2.MP, GND_ROTOR3.MP, IC2.GND, J2.1, J2.10, J2.13, J2.16, J2.19, J2.4, J2.7, J3.2, J4.1, J4.10, J4.4, J4.8, J4.9, R2.1, R3.1, SERVO_GND_CARG.MP, SERVO_GND_GAT.MP, SV1.14, SV1.20, SV1.25, SV1.34, SV1.39, SV1.6, SV1.9, U$1.1, U$1.10, U$1.15, U$1.18, U$1.21, U$1.24, U$1.27, U$1.30, U$1.4
- removed net N$10: C2.1, C3.1, U1.GND/ADJ
- new net 5V_CARCASA: 5V_CARCASA.MP, J4.1, J4.5, J4.6, J4.7
- new net GND_CARCASA: GND_CARCASA.MP, J4.10, J4.4, J4.8, J4.9
- new net GND_OPI: 10K_GND.2, C2.1, C3.1, C4.1, C5.1, GND_LIDAR.P, GND_OPI.MP, IC2.GND, J1.10, J1.5, J1.7, J2.1, J2.10, J2.13, J2.16, J2.19, J2.4, J2.7, R2.1, R3.1, SV1.14, SV1.20, SV1.25, SV1.34, SV1.39, SV1.6, SV1.9, U$1.1, U$1.10, U$1.15, U$1.18, U$1.21, U$1.24, U$1.27, U$1.30, U$1.4, U1.GND/ADJ
- new net GND_SERVOS: GND_SERVOS.MP, SERVO_GND_CARG.MP, SERVO_GND_GAT.MP
- new net LIGHTS_GND: LIGHTS_GND.MP
- new net N$2: J3.2
- net 5V_OPI: no longer J4.5, J4.6, J4.7
Other:
- note added: "Conector carcasa"
- moved on the sheet: 5V_OPI, 5V_SERVOS
