File: rotor_MCU/rotor_khamex_4.1_completo.brd (EAGLE design)
At the start: 156.5 x 131.5 mm, 38 parts, among them IC1 SN65HVD230DR, IC3 ELVX-L10D-HRRN-C-N2A4, J1 DF40C-80DS-0.4V(51)_ROWSWAP, J2 DF40C-80DS-0.4V(51)_ROWSWAP, J3 FTSH-110-01-F-DV, J4 612010235121, J5 612010235121, P2 686110188622, U1 LTC4368CMS-2#PBF

Commit message: Dani: paso a kicad
Parts:
- added CANH1, CANL1: LSP11, solpad:LSP11
- moved CANH 0.60 mm to (93.7, 18.5)
Connections:
- net CANH: now also CANH1.MP
- net CANL: now also CANL1.MP
Routing:
- net CANL: track 71.5 -> 318.1 mm, vias 0 -> 1
- net CANH: track 85.9 -> 325.4 mm
- net I2C0-SCL: track 259.8 -> 195.5 mm
- net 3V3-I2C: track 357.2 -> 315.9 mm
- net I2C0-SDA: track 208.1 -> 170.7 mm, vias 5 -> 4
- net GND: track 611.0 -> 576.7 mm
- net PWM9_SYNC: track 186.1 -> 166.8 mm, vias 2 -> 1
- net TCK/SWCLK: track 73.3 -> 75.7 mm
