File: rotor_MCU/rotor_khamex_4.1_completo.sch (EAGLE design)
At the start: 38 parts, among them IC1 SN65HVD230DR, IC3 ELVX-L10D-HRRN-C-N2A4, J1 DF40C-80DS-0.4V(51)_ROWSWAP, J2 DF40C-80DS-0.4V(51)_ROWSWAP, J3 FTSH-110-01-F-DV, J4 612010235121, J5 612010235121, P2 686110188622, U1 LTC4368CMS-2#PBF

Commit message: Dani: paso a kicad
Parts:
- added CANH1, CANL1: LSP11, solpad:LSP11
Connections:
- net CANH: now also CANH1.MP
- net CANL: now also CANL1.MP
Changed lines of the file:
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@@
 <part name="5V_ROTOR" library="solpad" deviceset="SE14" device=""/>
 <part name="GND" library="solpad" deviceset="SE14" device=""/>
+<part name="CANH1" library="solpad" deviceset="LSP11" device=""/>
+<part name="CANL1" library="solpad" deviceset="LSP11" device=""/>
 </parts>
 <sheets>
@@
 <instance part="GND22" gate="1" x="66.04" y="187.96" rot="R270"/>
 <instance part="GND23" gate="1" x="91.44" y="190.5" rot="R90"/>
+<instance part="CANH1" gate="1" x="350.52" y="48.26" rot="R270"/>
+<instance part="CANL1" gate="1" x="350.52" y="40.64" rot="R270"/>
 </instances>
 <busses>
@@
 <label x="60.96" y="190.5" size="0.8128" layer="95" rot="R180" xref="yes"/>
 </segment>
+<segment>
+<pinref part="CANH1" gate="1" pin="MP"/>
+<wire x1="347.98" y1="48.26" x2="342.9" y2="48.26" width="0.1524" layer="91"/>
+<label x="342.9" y="48.26" size="1.778" layer="95" rot="R180" xref="yes"/>
+</segment>
 </net>
 <net name="CANL" class="0">
@@
 <label x="96.52" y="187.96" size="0.8128" layer="95" xref="yes"/>
 </segment>
-</net>
+<segment>
+<pinref part="CANL1" gate="1" pin="MP"/>
+<wire x1="347.98" y1="40.64" x2="342.9" y2="40.64" width="0.1524" layer="91"/>
+<label x="342.9" y="40.64" size="1.778" layer="95" rot="R180" xref="yes"/>
+</segment>
+</net>
