File: rotor_MCU/rotor_khamex_4.5.brd (EAGLE design)
At the start: 156.5 x 131.5 mm, 40 parts, among them IC1 SN65HVD230DR, IC3 ELVX-L10D-HRRN-C-N2A4, J1 DF40C-80DS-0.4V(51)_ROWSWAP, J2 DF40C-80DS-0.4V(51)_ROWSWAP, J3 FTSH-110-01-F-DV, J4 612010235121, J5 612010235121, P2 686110188622, U1 LTC4368CMS-2#PBF

Commit message: actualizacion rotor
Parts:
- removed P2: 686110188622, 686110188622:686110188622
- added U$1, U$3, U$4, U$5, U$6, U$7: (no value), fiducial:CIRCLE-1MM-3R
- moved C4 133.2 mm to (-93.4, 64.7)
- moved LED1 133.2 mm to (-93.7, 69.4)
- moved MOSFET 133.2 mm to (-101.1, 82.8)
- moved R1 133.2 mm to (-106.6, 81.2)
- moved R10 133.2 mm to (-99.1, 70.0)
- moved R5 133.2 mm to (-107.0, 71.8)
- moved R6 133.2 mm to (-91.9, 77.7)
- moved R8 133.2 mm to (-107.1, 77.3)
- moved R9 133.2 mm to (-103.3, 70.1)
- moved U1 133.2 mm to (-101.3, 75.7)
- moved CANH 26.5 mm to (71.5, 10.6)
- moved BATT_- 25.3 mm to (52.7, 3.90)
- moved CANL 24.0 mm to (71.5, 7.90)
- moved SW_50V_OUT 7.60 mm to (154.3, 9.70)
- moved MODULO_GND_IN1 7.50 mm to (154.2, 2.00)
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Connections:
- removed net N$1: J1.22
- net GND: now also J1.22, J1.42, J1.47, J1.54, PIN1.4
Routing:
- net GND: track 677.7 -> 582.1 mm
- net PWM5: track 77.3 -> 166.8 mm, vias 0 -> 2
- net TMS/SWDIO: track 0.00 -> 65.2 mm, vias 0 -> 2
- net I2C0-SCL: track 229.9 -> 262.7 mm, vias 4 -> 2
- net I2C0-SDA: track 229.5 -> 261.5 mm, vias 4 -> 2
- net CAN1TX: track 102.8 -> 77.2 mm
- net CAN1RX: track 115.3 -> 98.5 mm, vias 4 -> 2
- net SDA: track 111.8 -> 122.6 mm
- net SCL: track 110.5 -> 118.0 mm
- net 3V3-I2C: track 302.4 -> 295.1 mm, vias 3 -> 4
- net TCK/SWCLK: track 69.0 -> 75.6 mm
- net 3V3: track 160.7 -> 155.5 mm
- net PWM9_SYNC: track 183.9 -> 178.7 mm, vias 3 -> 1
- net CANL: track 354.0 -> 348.9 mm, vias 3 -> 1
- net CANH: track 358.3 -> 353.2 mm
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- added copper zone on layer 2, net GND
Other:
- board size 156.5 x 131.5 mm -> 156.5 x 131.8 mm
- board text added: "K1_ROT_V0.1_rev4.5"
- board text removed: "330UF"
- board text removed: "BAT +"
- board text removed: "C1"
- board text removed: "K1_ROT_V0.1_rev4.0"
