File: rotor_MCU/rotor_khamex_4.5.sch (EAGLE design)
At the start: 40 parts, among them IC1 SN65HVD230DR, IC3 ELVX-L10D-HRRN-C-N2A4, J1 DF40C-80DS-0.4V(51)_ROWSWAP, J2 DF40C-80DS-0.4V(51)_ROWSWAP, J3 FTSH-110-01-F-DV, J4 612010235121, J5 612010235121, P2 686110188622, U1 LTC4368CMS-2#PBF

Commit message: actualizacion rotor
Parts:
- removed P2: 686110188622, 686110188622:686110188622
Connections:
- removed net N$1: J1.22
- net GND: now also J1.22, J1.42, J1.47, J1.54, PIN1.4
Other:
- note removed: "Conector datos rotor (Mierdiflex)"
- moved on the sheet: J1, J2
