File: rotor_MCU/rotor_khamex_4.6.sch (EAGLE design)
At the start: 39 parts, among them IC1 SN65HVD230DR, IC3 ELVX-L10D-HRRN-C-N2A4, J1 DF40C-80DS-0.4V(51)_ROWSWAP, J2 DF40C-80DS-0.4V(51)_ROWSWAP, J3 FTSH-110-01-F-DV, J4 612010235121, J5 612010235121, U1 LTC4368CMS-2#PBF

Commit message: JC: Cambios en zenit y rotor
Parts:
- removed C4: 100nF, eagle-ltspice:C
- removed J5: 612010235121, Eagle_WR-BHD_rev24a:6120XX235121_612010235121
- removed LED1: (no value), led:LED
- removed MOSFET: AO4407A, AO4407A:AO4407A
- removed R1: 1.1M, eagle-ltspice:R
- removed R10, R5: 10k, eagle-ltspice:R
- removed R6: 100, eagle-ltspice:R
- removed R8: 22k, eagle-ltspice:R
- removed R9: 787k, eagle-ltspice:R
- removed U1: LTC4368CMS-2#PBF, LTC4368CMS-2_PBF:LTC4368CMS-2#PBF
Connections:
- removed net GATE_PWR: MOSFET.G, R6.1
- removed net N$11: R5.2, R9.1, U1.UV
- removed net N$12: R1.1, R10.2, U1.OV
- removed net N$13: LED1.C, R8.2
- removed net N$14: R6.2, U1.GATE
- removed net N$2: LED1.A, U1.!FAULT
- removed net N$20: U1.RETRY
- removed net N$21: U1.GND
- removed net VBAT: MOSFET.D, U1.SENSE, U1.VOUT
- removed net VBAT_RAW: C4.2, MOSFET.S, R1.2, R8.1, R9.2, U1.!SHDN, U1.VIN
- net CANH: no longer J5.9
- net CANL: no longer J5.8
- net GND: no longer J5.10, J5.5, J5.7
- net PWM5: no longer J5.4
- net PWM9_SYNC: no longer J5.6
Other:
- note removed: "CONTROL VOLTAJE BATERÍA"
- moved on the sheet: J4
